Commit message: feat: Add depth camera and launch file for RTAB-Map
Add RGBD camera to my_robot.xacro and my_robot.gazebo, and
add mapping.launch file to launch RTAB-Map node

File: src/my_robot/urdf/my_robot.xacro (robot description, xacro)
@@ -186,3 +186,10 @@
     <child link="hokuyo" />
   </joint>
+  <joint name="camera_optical_joint" type="fixed">
+    <origin xyz="0 0 0" rpy="-1.5707 0 -1.5707"/>
+    <parent link="camera"/>
+    <child link="camera_link_optical"/>
+  </joint>
+  <link name="camera_link_optical">
+  </link>
 </robot>
